File: PCB/ISO7816/ISO7816.kicad_pcb (KiCad board)
At the start: 2 copper layers, 68 x 81 mm, 48 parts, among them J1 Conn_01x02, J3 Conn_01x08, J4 Conn_01x08, J6 USB-C-Socket-H, J7 TC2030-USB-NL-DS, Q1 BSS138PS, Q2 BSS138PS, Q3 BSS138PS, U1 ESP32-S3-MINI-1-N4R2, U2 TPS562246, U4 TPS22916CNYFPR, U5 TPS22916CNYFPR

Commit message: Schematic
Parts:
- removed C1, C9: C, RevK:C_0805
- removed C10, C11, C12, C13, C14, C7, C8: C, RevK:C_0201
- removed C2, C3, C4: C, RevK:C_0402
- removed C5: C, RevK:C_0603
- removed D4: ~, RevK:DFN1006-2L
- removed L1: L, RevK:L_5x5
- removed R7: R, RevK:R_0201
- added C15: 22uF 25V, RevK:C_0805, F.Cu at (182.0, 91.0)
- added C16: 100nF 25V, RevK:C_0402, F.Cu at (182.5, 93.5)
- added C17: 100nF 25V, RevK:C_0402, F.Cu at (182.5, 94.5)
- added C18: 100nF, RevK:C_0201, F.Cu at (177.4, 95.0)
- added C19: 18pF, RevK:C_0201, F.Cu at (178.6, 95.0)
- added C20: 47uF 6V, RevK:C_0805, F.Cu at (173.5, 86.0)
- added C21: 100nF, RevK:C_0201, F.Cu at (173.5, 89.1)
- added C22: 100nF, RevK:C_0201, F.Cu at (161.1, 106.9)
- added C23: 100nF, RevK:C_0201, F.Cu at (156.7, 99.6)
- added C24: 100nF, RevK:C_0201, F.Cu at (173.5, 87.4)
- added C25: 100nF, RevK:C_0201, F.Cu at (173.5, 88.3)
- added L2: 4.7uH, RevK:L_5x5, F.Cu at (178.0, 88.0)
- added Q4: BSS84, Package_TO_SOT_SMD:SOT-23, F.Cu at (156.0, 87.5)
- added R14: 150k 1%, RevK:R_0201, F.Cu at (178.0, 95.0)
- added R15: 150k 1%, RevK:R_0201, F.Cu at (179.2, 95.0)
- added R16: 33k 1%, RevK:R_0201, F.Cu at (179.8, 95.0)
- added R17: 10k, RevK:R_0201, F.Cu at (151.2, 88.8)
- added R18: 10k, RevK:R_0201, F.Cu at (153.5, 95.7)
- added R19: 10k, RevK:R_0201, F.Cu at (153.5, 91.6)
- added R20: 10R, RevK:R_0201, F.Cu at (152.2, 93.8)
- added U3: TPS562246, RevK:SOT-563, F.Cu at (178.0, 93.0)
- added U6: SN74LVC1T45DCK, Package_TO_SOT_SMD:SOT-363_SC-70-6, F.Cu at (154.6, 97.3)
- C6: value C -> 1uF; footprint RevK:C_0402 -> RevK:C_0201
- R1: value R -> 20k
- R12, R13: value 1k -> 10k
- R2: value R -> 10k; footprint RevK:R_0402 -> RevK:R_0201
- R3, R4: value R -> 10k
- U2: value TPS562246 -> SN74LVC1T45DCK; footprint RevK:SOT-563 -> Package_TO_SOT_SMD:SOT-363_SC-70-6
- moved C6 45.5 mm to (202.8, 98.5), turned to 180 degrees
- moved D1 38.6 mm to (203.0, 78.0), turned to 180 degrees
- moved R13 35.4 mm to (159.5, 108.1), turned to 180 degrees
- moved R12 35.3 mm to (159.5, 104.6), turned to 180 degrees
- moved R4 34.8 mm to (149.4, 83.3)
- moved R1 32.3 mm to (153.5, 86.0), turned to 180 degrees
- moved U5 31.6 mm to (159.5, 107.0), turned to 180 degrees
- moved U4 31.6 mm to (159.5, 103.5), turned to 180 degrees
- moved R2 22.7 mm to (204.0, 98.5), turned to 180 degrees
- moved D6 22.5 mm to (147.8, 84.6), turned to -90 degrees
- moved U2 21.9 mm to (154.4, 93.4), turned to 180 degrees
- moved Q1 19.2 mm to (154.5, 103.8), turned to 180 degrees
- moved R9 18.6 mm to (147.8, 86.0), turned to -90 degrees
- moved D2 17.8 mm to (156.7, 102.7), turned to -90 degrees
- moved R10 15.5 mm to (184.1, 77.8), turned to 90 degrees
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Connections:
- D3 pad 2: Net-(Q1B-GP) -> Net-(U2-B)
- D5 pad 2: Net-(Q2B-GP) -> Net-(U6-B)
- D6 pad 2: Net-(Q3A-GN) -> Net-(Q2A-GN)
- Q2 pad 3: C_CLK_I -> unconnected-(Q2B-SP-Pad3)
- Q2 pad 4: GND -> unconnected-(Q2B-DP-Pad4)
- Q2 pad 5: Net-(Q2B-GP) -> unconnected-(Q2B-GP-Pad5)
- Q2 pad 6: C_RST_I -> C_I/O_I
- Q3 pad 2: Net-(Q3A-GN) -> C_I/O_E
- Q3 pad 3: (no net) -> C_I/O
- Q3 pad 4: (no net) -> GND
- Q3 pad 5: (no net) -> C_I/O_O
- Q3 pad 6: C_I/O_I -> Net-(Q3A-DN)
- R1 pad 1: EN -> Net-(Q4-D)
- R1 pad 2: VBUS -> C_I/O
- R3 pad 1: +3.3V -> Net-(Q3A-DN)
- R3 pad 2: FB -> C_VCC
- R4 pad 1: FB -> GND
- R4 pad 2: GND -> C_I/O_E
- R8 pad 1: Net-(Q2B-GP) -> Net-(U6-B)
- R9 pad 1: Net-(Q3A-GN) -> Net-(Q2A-GN)
- U1 pad 22: unconnected-(U1-GPIO18-Pad22) -> C_INSERT
- U1 pad 27: LED -> unconnected-(U1-GPIO47-Pad27)
- U1 pad 28: unconnected-(U1-GPIO33-Pad28) -> C_I/O_I
- U1 pad 29: RX -> C_I/O_E
- U1 pad 30: TX -> unconnected-(U1-GPIO48-Pad30)
- U1 pad 31: RX2 -> C_I/O_O
- U1 pad 32: TX2 -> C_RST_IO
- U1 pad 33: unconnected-(U1-GPIO37-Pad33) -> C_RST_E
- U1 pad 34: unconnected-(U1-GPIO38-Pad34) -> C_CLK_IO
- U1 pad 35: unconnected-(U1-GPIO39-Pad35) -> C_CLK_E
- U1 pad 36: unconnected-(U1-GPIO40-Pad36) -> C_VCC_I
- U1 pad 37: unconnected-(U1-GPIO41-Pad37) -> C_VPP_I
- U1 pad 38: unconnected-(U1-GPIO42-Pad38) -> C_5V
- U1 pad 41: unconnected-(U1-GPIO45-Pad41) -> C_3V3
- U1 pad 5: unconnected-(U1-GPIO1-Pad5) -> LED
- U2 pad 1: VBUS -> +3.3V
- U2 pad 2: SW -> GND
- U2 pad 3: GND -> C_RST_IO
- U2 pad 4: BST -> Net-(U2-B)
- U2 pad 5: EN -> C_RST_E
- U2 pad 6: FB -> C_VCC
Routing:
- net +3.3V: track 0.00 -> 147.1 mm, vias 0 -> 7
- net C_I/O: track 78.8 -> 168.1 mm
- net VBUS: track 0.00 -> 80.1 mm
- net C_VCC: track 91.5 -> 160.9 mm, vias 2 -> 3
- net C_VPP: track 78.1 -> 145.1 mm
- net C_8: track 82.5 -> 138.3 mm
- net C_I/O_E: track 0.00 -> 55.2 mm, vias 0 -> 2
- net C_CLK_E: track 0.00 -> 50.8 mm, vias 0 -> 2
- net C_VCC_I: track 0.00 -> 50.1 mm, vias 0 -> 2
- net C_RST_E: track 0.00 -> 49.6 mm, vias 0 -> 2
- net D-: track 0.00 -> 49.2 mm, vias 0 -> 3
- net C_I/O_O: track 0.00 -> 49.1 mm, vias 0 -> 2
- net C_I/O_I: track 0.00 -> 48.2 mm, vias 0 -> 2
- net C_3V3: track 0.00 -> 47.9 mm, vias 0 -> 2
- net C_VPP_I: track 0.00 -> 47.7 mm, vias 0 -> 2
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- added copper zone on F.Cu, net VBUS
Other:
- board text added: "1"
- board text added: "33 34 35 36 37 38 39 40 41 42 45 18"
- board text added: "A"
- board text added: "C_I/O_I C_I/O_E C_I/O_O C_RST_IO C_RST_E C_CLK_IO C_CLK_E C_VCC_I C_VPP_I C_5V C_3V3 C_INSERT"
- board text added: "GND"
- board text added: "I/O_E Enables 20k pull up so I/O_O can pull down RST_E and CLK_E enables level shifter output for RST_IO & CLK_IO _I are inputs 5V/3V3 Apply power to VCC Card inserted"
- board text added: "LED"
- board text added: "Reader Emulator Monitor"
- board text added: "VCC RST CLK C4 GND VPP I/O C8"
