File: PCB/ISO7816/ISO7816.kicad_pcb (KiCad board)
At the start: 2 copper layers, 68 x 81 mm, 54 parts, among them J1 Conn_01x02, J3 Conn_01x08, J4 Conn_01x08, J6 USB-C-Socket-H, J7 TC2030-USB-NL-DS, Q1 BSS138PS, Q2 BSS138PS, Q3 BSS138PS, Q4 BSS84, U1 ESP32-S3-MINI-1-N4R2, U2 SN74LVC1T45DCK, U3 TPS562246, U4 TPS22916CNYFPR, U5 TPS22916CNYFPR, U6 SN74LVC1T45DCK

Commit message: Ready to order
Parts:
- moved C21 17.4 mm to (156.7, 93.7), turned to -90 degrees
- moved C25 0.85 mm to (173.8, 87.5)
- turned J1 to 180 degrees
Routing:
- net VBUS: track 80.1 -> 85.7 mm
- net D-: track 49.2 -> 44.5 mm
- net +3.3V: track 147.1 -> 151.2 mm
- net D+: track 46.5 -> 43.8 mm
- net Net-(J1-Pin_2): track 10.1 -> 7.74 mm
- net C_INSERT: track 29.1 -> 28.5 mm
Other:
- board text added: "0"
- board text added: "Designed by RevK www.me.uk toot.me.uk/@RevK"
- board text added: "®"
